File: dynamixel.kicad_sch (KiCad schematic)
At the start: 17 parts, among them J5 Conn_01x03_Pin, J9 Conn_01x03_Pin, Q6 BSS138, Q7 BSS138, Q8 BSS138, U7 74LVC2G241

Commit message: Fixing 10K Part Number
Parts:
- R19, R22, R24, R25, R26, R28, R29: JLCPCB C17414 -> C25744
Changed lines of the file:
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@@
 			)
 		)
-		(property "JLCPCB" "C17414"
+		(property "JLCPCB" "C25744"
 			(at 107.95 78.74 0)
 			(effects
@@
 			)
 		)
-		(property "JLCPCB" "C17414"
+		(property "JLCPCB" "C25744"
 			(at 60.96 62.23 0)
 			(effects
@@
 			)
 		)
-		(property "JLCPCB" "C17414"
+		(property "JLCPCB" "C25744"
 			(at 90.17 78.74 0)
 			(effects
@@
 			)
 		)
-		(property "JLCPCB" "C17414"
+		(property "JLCPCB" "C25744"
 			(at 162.56 49.53 0)
 			(effects
@@
 			)
 		)
-		(property "JLCPCB" "C17414"
+		(property "JLCPCB" "C25744"
 			(at 97.79 49.53 0)
 			(effects
@@
 			)
 		)
-		(property "JLCPCB" "C17414"
+		(property "JLCPCB" "C25744"
 			(at 78.74 62.23 0)
 			(effects
@@
 			)
 		)
-		(property "JLCPCB" "C17414"
+		(property "JLCPCB" "C25744"
 			(at 121.92 49.53 0)
 			(effects
