File: charge_bay.kicad_pcb (KiCad board)
At the start: 4 copper layers, 90 x 51.4 mm, 111 parts, among them J1 USB_C_Receptacle_USB2.0, J10 Conn_01x03_Pin, J11 Conn_01x05_Socket, J2 Screw_Terminal_01x04, J3 Conn_01x03_Pin, J4 Conn_01x03_Pin, J5 Conn_01x03_Pin, J6 Conn_01x05_Socket, J7 Screw_Terminal_01x04, J8 Conn_01x03_Pin, J9 Conn_01x03_Pin, Q1 MMBT3904, Q2 MMBT3904, Q3 MMBT3904, Q4 MMBT3904, Q5 MMBT3904, Q6 BSS138, Q7 BSS138, Q8 BSS138, SW1 SW_Push, SW2 SW_Push, U1 RP2040, U2 W25Q16JVUXIQ TR, U4 LP38691SD-3.3, U5 MCP2515-xST, U6 TJA1051T-3, U7 74LVC2G241, Y1 Crystal_GND24, Y2 ABM8-272-T3

Commit message: Feature/release upload (#1)
* Adding Release Artifact Capability

* Update to KiCad 9

* Further Release Process Updates

- try to fix component warnings by syncing to schematic
- add auto version updates to PCB tagging
- adjust the URL on the board to point to the correct repo.
Other:
- board text added: "<<version>> - <<hash>>"
- board text added: "http://bitbucket.org/daveismith/charge-bay"
- board text removed: "http://bitbucket.org/daveismith/hardware"
- board text removed: "v1.0 - <<hash>>"
